File: CogLightBadgeTHT.sch (KiCad schematic (older format))
At the start: 28 parts, among them J1 AVR-ISP, SW1 SW_SPDT, SW2 SW_Push, SW3 SW_Push, U1 ATtiny84A-PU

Commit message: Downsized pcb and component layout
Parts:
- added C1: 100nF, Capacitor_THT:C_Disc_D5.0mm_W2.5mm_P5.00mm, symbol Device:C
Connections:
- net GND: now also C1.2
- net VCC: now also C1.1
Changed lines of the file:
@@
+	1    0    0    -1
+$EndComp
+$Comp
+L Device:C C1
+U 1 1 601B337A
+P 2850 1800
+F 0 "C1" H 2965 1846 50  0000 L CNN
+F 1 "100nF" H 2965 1755 50  0000 L CNN
+F 2 "Capacitor_THT:C_Disc_D5.0mm_W2.5mm_P5.00mm" H 2888 1650 50  0001 C CNN
+F 3 "~" H 2850 1800 50  0001 C CNN
+	1    2850 1800
+	1    0    0    -1
+$EndComp
+$Comp
+L power:VCC #PWR0111
+U 1 1 601B3DA6
+P 2850 1650
+F 0 "#PWR0111" H 2850 1500 50  0001 C CNN
+F 1 "VCC" H 2865 1823 50  0000 C CNN
+F 2 "" H 2850 1650 50  0001 C CNN
+F 3 "" H 2850 1650 50  0001 C CNN
+	1    2850 1650
+	1    0    0    -1
+$EndComp
+$Comp
+L power:GND #PWR0112
+U 1 1 601B44CA
+P 2850 1950
+F 0 "#PWR0112" H 2850 1700 50  0001 C CNN
+F 1 "GND" H 2855 1777 50  0000 C CNN
+F 2 "" H 2850 1950 50  0001 C CNN
+F 3 "" H 2850 1950 50  0001 C CNN
+	1    2850 1950
 	1    0    0    -1
 $EndComp

Commit message: Improved siklscreen layout
Parts:
- C1: value 100nF -> .1uF
Changed lines of the file:
@@
 P 2850 1800
 F 0 "C1" H 2965 1846 50  0000 L CNN
-F 1 "100nF" H 2965 1755 50  0000 L CNN
+F 1 ".1uF" H 2965 1755 50  0000 L CNN
 F 2 "Capacitor_THT:C_Disc_D5.0mm_W2.5mm_P5.00mm" H 2888 1650 50  0001 C CNN
 F 3 "~" H 2850 1800 50  0001 C CNN

Commit message: Changing LED resistors to 330 ohm
Parts:
- R1, R2, R3, R4: value 1k -> 330
Changed lines of the file:
@@
 P 1650 3500
 F 0 "R1" V 1443 3500 50  0000 C CNN
-F 1 "1k" V 1534 3500 50  0000 C CNN
+F 1 "330" V 1534 3500 50  0000 C CNN
 F 2 "Resistor_THT:R_Axial_DIN0207_L6.3mm_D2.5mm_P7.62mm_Horizontal" V 1580 3500 50  0001 C CNN
 F 3 "~" H 1650 3500 50  0001 C CNN
@@
 P 1650 4500
 F 0 "R2" V 1443 4500 50  0000 C CNN
-F 1 "1k" V 1534 4500 50  0000 C CNN
+F 1 "330" V 1534 4500 50  0000 C CNN
 F 2 "Resistor_THT:R_Axial_DIN0207_L6.3mm_D2.5mm_P7.62mm_Horizontal" V 1580 4500 50  0001 C CNN
 F 3 "~" H 1650 4500 50  0001 C CNN
@@
 P 1650 5500
 F 0 "R3" V 1443 5500 50  0000 C CNN
-F 1 "1k" V 1534 5500 50  0000 C CNN
+F 1 "330" V 1534 5500 50  0000 C CNN
 F 2 "Resistor_THT:R_Axial_DIN0207_L6.3mm_D2.5mm_P7.62mm_Horizontal" V 1580 5500 50  0001 C CNN
 F 3 "~" H 1650 5500 50  0001 C CNN
@@
 P 1650 6500
 F 0 "R4" V 1443 6500 50  0000 C CNN
-F 1 "1k" V 1534 6500 50  0000 C CNN
+F 1 "330" V 1534 6500 50  0000 C CNN
 F 2 "Resistor_THT:R_Axial_DIN0207_L6.3mm_D2.5mm_P7.62mm_Horizontal" V 1580 6500 50  0001 C CNN
 F 3 "~" H 1650 6500 50  0001 C CNN
